Commit message: Fixed

File: isaacsim/urdf/base_link_description/urdf/base_link.urdf (robot description, URDF)
Before this commit: robot base_link, 1 links, 0 joints
Links:
- link base_link: geometry collision mesh filename=./urdf/base_link_description/meshes/base_link.stl scale=0.001 0.001 0.001; visual mesh filename=./urdf/base_link_description/meshes/base_link.stl scale=0.001 0.001 0.001

File: isaacsim/urdf/box_obstacle_description/urdf/box_obstacle.urdf (robot description, URDF)
Before this commit: robot base_link, 1 links, 0 joints
Links:
- link base_link: geometry collision mesh filename=./urdf/box_obstacle_description/meshes/base_link.stl scale=0.001 0.001 0.001; visual mesh filename=./urdf/box_obstacle_description/meshes/base_link.stl scale=0.001 0.001 0.001
